File: bumps.sch (KiCad schematic (older format))
At the start: 22 parts

Commit message: o Add step/dir signals.
Parts:
- gave numbers to parts that had none: 22
Connections:
- net labels added: DIR_A, DIR_B, DIR_C, DIR_E, DIR_U, DIR_X, DIR_Y, DIR_Z, STEP_A, STEP_B, STEP_C, STEP_E, STEP_U, STEP_Y, STEP_Z
- wire segments 74 -> 59

Commit message: added bumps.mod footprints file and set footprints in schematic
Parts:
- P1, P2, P5, P6, P7: footprint (none) -> pin_array_3x2
- P10, P11, P12, P3, P4: footprint (none) -> pin_array_4x2
- P8, P9: footprint MODULE -> PIN_ARRAY_23X2
- R1, R2, R3, R4, R5: footprint (none) -> SM0805
- U1, U2, U3, U4, U5: footprint MODULE -> POLOLU
Changed lines of the file:
@@
-EESchema Schematic File Version 2
+EESchema Schematic File Version 2  date Sat 01 Feb 2014 09:23:24 PM PST
 LIBS:power
 LIBS:device
@@
 LIBS:valves
 LIBS:BUMPS
-EELAYER 24 0
+EELAYER 27 0
 EELAYER END
 $Descr A4 11693 8268
@@
 F 0 "U1" H 3800 4300 50  0000 C CNN
 F 1 "POLOLUSTEPPER" H 3800 4800 50  0000 C CNN
-F 2 "MODULE" H 3850 4700 50  0001 C CNN
+F 2 "POLOLU" H 3850 4700 50  0001 C CNN
 F 3 "DOCUMENTATION" H 3800 3800 50  0001 C CNN
 	1    3800 4300
@@
 F 0 "P8" H 5300 2950 50  0000 C CNN
 F 1 "bbbp8" H 5300 3050 50  0000 C CNN
-F 2 "MODULE" H 5300 3100 50  0001 C CNN
+F 2 "PIN_ARRAY_23X2" H 5300 3100 50  0001 C CNN
 F 3 "DOCUMENTATION" H 5300 600 50  0001 C CNN
 	1    5300 1850
@@
 F 0 "P9" H 2350 2650 50  0000 C CNN
 F 1 "bbbp9" H 2350 900 50  0000 C CNN
-F 2 "MODULE" H 2350 2800 50  0001 C CNN
+F 2 "PIN_ARRAY_23X2" H 2350 2800 50  0001 C CNN
 F 3 "DOCUMENTATION" H 2350 350 50  0001 C CNN
 	1    2350 1700
@@
 F 0 "#PWR01" H 3650 800 30  0001 C CNN
 F 1 "GND" H 3650 730 30  0001 C CNN
-F 2 "" H 3650 800 60  0000 C CNN
-F 3 "" H 3650 800 60  0000 C CNN
 	1    3650 800
 	1    0    0    -1
@@
 F 0 "#PWR02" H 1000 800 30  0001 C CNN
 F 1 "GND" H 1000 730 30  0001 C CNN
-F 2 "" H 1000 800 60  0000 C CNN
-F 3 "" H 1000 800 60  0000 C CNN
 	1    1000 800
 	1    0    0    -1
@@
 F 0 "#PWR03" H 4550 750 30  0001 C CNN
 F 1 "GND" H 4550 680 30  0001 C CNN
-F 2 "" H 4550 750 60  0000 C CNN
-F 3 "" H 4550 750 60  0000 C CNN
 	1    4550 750
 	1    0    0    -1
@@
 F 0 "#PWR04" H 6050 750 30  0001 C CNN
 F 1 "GND" H 6050 680 30  0001 C CNN
-F 2 "" H 6050 750 60  0000 C CNN
-F 3 "" H 6050 750 60  0000 C CNN
 	1    6050 750
 	1    0    0    -1
@@
 F 0 "#PWR05" H 4550 4700 30  0001 C CNN
 F 1 "GND" H 4550 4630 30  0001 C CNN
-F 2 "" H 4550 4700 60  0000 C CNN
-F 3 "" H 4550 4700 60  0000 C CNN
 	1    4550 4700
 	1    0    0    -1
@@
 F 0 "#PWR06" H 4550 4050 30  0001 C CNN
 F 1 "GND" H 4550 3980 30  0001 C CNN
-F 2 "" H 4550 4050 60  0000 C CNN
-F 3 "" H 4550 4050 60  0000 C CNN
 	1    4550 4050
 	1    0    0    -1
@@
 F 0 "P3" H 4950 4550 50  0000 C CNN
 F 1 "CONN_4X2" V 4950 4300 40  0000 C CNN
-F 2 "" H 4950 4300 60  0000 C CNN
-F 3 "" H 4950 4300 60  0000 C CNN
+F 2 "pin_array_4x2" V 5050 4300 40  0001 C CNN
 	1    4950 4300
 	1    0    0    -1
@@
 F 0 "P1" H 2250 4450 50  0000 C CNN
 F 1 "CONN_3X2" V 2250 4250 40  0000 C CNN
-F 2 "" H 2250 4200 60  0000 C CNN
-F 3 "" H 2250 4200 60  0000 C CNN
+F 2 "pin_array_3x2" V 2350 4250 40  0001 C CNN
 	1    2250 4200
 	1    0    0    -1
@@
 F 0 "R1" V 2530 4650 40  0000 C CNN
 F 1 "R" V 2457 4651 40  0000 C CNN
-F 2 "" V 2380 4650 30  0000 C CNN
-F 3 "" H 2450 4650 30  0000 C CNN
+F 2 "SM0805" V 2380 4650 30  0001 C CNN
 	1    2450 4650
 	-1   0    0    1
@@
 F 0 "#PWR07" H 2450 4900 30  0001 C CNN
 F 1 "GND" H 2450 4830 30  0001 C CNN
-F 2 "" H 2450 4900 60  0000 C CNN
-F 3 "" H 2450 4900 60  0000 C CNN
 	1    2450 4900
 	1    0    0    -1
@@
 F 0 "U5" H 9200 4800 50  0000 C CNN
 F 1 "POLOLUSTEPPER" H 9200 5300 50  0000 C CNN
-F 2 "MODULE" H 9250 5200 50  0001 C CNN
+F 2 "POLOLU" H 9250 5200 50  0001 C CNN
 F 3 "DOCUMENTATION" H 9200 4300 50  0001 C CNN
 	1    9200 4800
@@
 F 0 "#PWR08" H 9950 5200 30  0001 C CNN
 F 1 "GND" H 9950 5130 30  0001 C CNN
-F 2 "" H 9950 5200 60  0000 C CNN
-F 3 "" H 9950 5200 60  0000 C CNN
 	1    9950 5200
 	1    0    0    -1
@@
 F 0 "#PWR09" H 9950 4550 30  0001 C CNN
 F 1 "GND" H 9950 4480 30  0001 C CNN
-F 2 "" H 9950 4550 60  0000 C CNN
-F 3 "" H 9950 4550 60  0000 C CNN
 	1    9950 4550
 	1    0    0    -1
@@
 F 0 "P10" H 10350 5050 50  0000 C CNN
 F 1 "CONN_4X2" V 10350 4800 40  0000 C CNN
-F 2 "" H 10350 4800 60  0000 C CNN
-F 3 "" H 10350 4800 60  0000 C CNN
+F 2 "pin_array_4x2" V 10450 4800 40  0001 C CNN
 	1    10350 4800
 	1    0    0    -1
@@
 F 0 "P7" H 7650 4950 50  0000 C CNN
 F 1 "CONN_3X2" V 7650 4750 40  0000 C CNN
-F 2 "" H 7650 4700 60  0000 C CNN
-F 3 "" H 7650 4700 60  0000 C CNN
+F 2 "pin_array_3x2" V 7750 4750 40  0001 C CNN
 	1    7650 4700
 	1    0    0    -1
@@
 F 0 "R5" V 7930 5150 40  0000 C CNN
 F 1 "R" V 7857 5151 40  0000 C CNN
-F 2 "" V 7780 5150 30  0000 C CNN
-F 3 "" H 7850 5150 30  0000 C CNN
+F 2 "SM0805" V 7780 5150 30  0001 C CNN
 	1    7850 5150
 	-1   0    0    1
@@
 F 0 "#PWR010" H 7850 5400 30  0001 C CNN
 F 1 "GND" H 7850 5330 30  0001 C CNN
-F 2 "" H 7850 5400 60  0000 C CNN
-F 3 "" H 7850 5400 60  0000 C CNN
 	1    7850 5400
 	1    0    0    -1
@@
 F 0 "U3" H 9200 1550 50  0000 C CNN
 F 1 "POLOLUSTEPPER" H 9200 2050 50  0000 C CNN
-F 2 "MODULE" H 9250 1950 50  0001 C CNN
+F 2 "POLOLU" H 9250 1950 50  0001 C CNN
 F 3 "DOCUMENTATION" H 9200 1050 50  0001 C CNN
 	1    9200 1550
@@
 F 0 "#PWR011" H 9950 1950 30  0001 C CNN
 F 1 "GND" H 9950 1880 30  0001 C CNN
-F 2 "" H 9950 1950 60  0000 C CNN
-F 3 "" H 9950 1950 60  0000 C CNN
 	1    9950 1950
 	1    0    0    -1
@@
 F 0 "#PWR012" H 9950 1300 30  0001 C CNN
 F 1 "GND" H 9950 1230 30  0001 C CNN
-F 2 "" H 9950 1300 60  0000 C CNN
-F 3 "" H 9950 1300 60  0000 C CNN
 	1    9950 1300
 	1    0    0    -1
@@
 F 0 "P11" H 10350 1800 50  0000 C CNN
 F 1 "CONN_4X2" V 10350 1550 40  0000 C CNN
-F 2 "" H 10350 1550 60  0000 C CNN
-F 3 "" H 10350 1550 60  0000 C CNN
+F 2 "pin_array_4x2" V 10450 1550 40  0001 C CNN
 	1    10350 1550
 	1    0    0    -1
@@
 F 0 "P5" H 7650 1700 50  0000 C CNN
 F 1 "CONN_3X2" V 7650 1500 40  0000 C CNN
-F 2 "" H 7650 1450 60  0000 C CNN
-F 3 "" H 7650 1450 60  0000 C CNN
+F 2 "pin_array_3x2" V 7750 1500 40  0001 C CNN
 	1    7650 1450
 	1    0    0    -1
@@
 F 0 "R3" V 7930 1900 40  0000 C CNN
 F 1 "R" V 7857 1901 40  0000 C CNN
-F 2 "" V 7780 1900 30  0000 C CNN
-F 3 "" H 7850 1900 30  0000 C CNN
+F 2 "SM0805" V 7780 1900 30  0001 C CNN
 	1    7850 1900
 	-1   0    0    1
@@
 F 0 "#PWR013" H 7850 2150 30  0001 C CNN
 F 1 "GND" H 7850 2080 30  0001 C CNN
-F 2 "" H 7850 2150 60  0000 C CNN
-F 3 "" H 7850 2150 60  0000 C CNN
 	1    7850 2150
 	1    0    0    -1
@@
 F 0 "U4" H 9200 3200 50  0000 C CNN
 F 1 "POLOLUSTEPPER" H 9200 3700 50  0000 C CNN
-F 2 "MODULE" H 9250 3600 50  0001 C CNN
+F 2 "POLOLU" H 9250 3600 50  0001 C CNN
 F 3 "DOCUMENTATION" H 9200 2700 50  0001 C CNN
 	1    9200 3200
@@
 F 0 "#PWR014" H 9950 3600 30  0001 C CNN
 F 1 "GND" H 9950 3530 30  0001 C CNN
-F 2 "" H 9950 3600 60  0000 C CNN
-F 3 "" H 9950 3600 60  0000 C CNN
 	1    9950 3600
 	1    0    0    -1
@@
 F 0 "#PWR015" H 9950 2950 30  0001 C CNN
 F 1 "GND" H 9950 2880 30  0001 C CNN
-F 2 "" H 9950 2950 60  0000 C CNN
-F 3 "" H 9950 2950 60  0000 C CNN
 	1    9950 2950
 	1    0    0    -1
@@
 F 0 "P12" H 10350 3450 50  0000 C CNN
 F 1 "CONN_4X2" V 10350 3200 40  0000 C CNN
-F 2 "" H 10350 3200 60  0000 C CNN
-F 3 "" H 10350 3200 60  0000 C CNN
+F 2 "pin_array_4x2" V 10450 3200 40  0001 C CNN
 	1    10350 3200
 	1    0    0    -1
@@
 F 0 "P6" H 7650 3350 50  0000 C CNN
 F 1 "CONN_3X2" V 7650 3150 40  0000 C CNN
-F 2 "" H 7650 3100 60  0000 C CNN
-F 3 "" H 7650 3100 60  0000 C CNN
+F 2 "pin_array_3x2" V 7750 3150 40  0001 C CNN
 	1    7650 3100
 	1    0    0    -1
@@
 F 0 "R4" V 7930 3550 40  0000 C CNN
 F 1 "R" V 7857 3551 40  0000 C CNN
-F 2 "" V 7780 3550 30  0000 C CNN
-F 3 "" H 7850 3550 30  0000 C CNN
+F 2 "SM0805" V 7780 3550 30  0001 C CNN
 	1    7850 3550
 	-1   0    0    1
@@
 F 0 "#PWR016" H 7850 3800 30  0001 C CNN
 F 1 "GND" H 7850 3730 30  0001 C CNN
-F 2 "" H 7850 3800 60  0000 C CNN
-F 3 "" H 7850 3800 60  0000 C CNN
 	1    7850 3800
 	1    0    0    -1
@@
 F 0 "U2" H 3800 6050 50  0000 C CNN
 F 1 "POLOLUSTEPPER" H 3800 6550 50  0000 C CNN
-F 2 "MODULE" H 3850 6450 50  0001 C CNN
+F 2 "POLOLU" H 3850 6450 50  0001 C CNN
 F 3 "DOCUMENTATION" H 3800 5550 50  0001 C CNN
 	1    3800 6050
@@
 F 0 "#PWR017" H 4550 6450 30  0001 C CNN
 F 1 "GND" H 4550 6380 30  0001 C CNN
-F 2 "" H 4550 6450 60  0000 C CNN
-F 3 "" H 4550 6450 60  0000 C CNN
 	1    4550 6450
 	1    0    0    -1
@@
 F 0 "#PWR018" H 4550 5800 30  0001 C CNN
 F 1 "GND" H 4550 5730 30  0001 C CNN
-F 2 "" H 4550 5800 60  0000 C CNN
-F 3 "" H 4550 5800 60  0000 C CNN
 	1    4550 5800
 	1    0    0    -1
@@
 F 0 "P4" H 4950 6300 50  0000 C CNN
 F 1 "CONN_4X2" V 4950 6050 40  0000 C CNN
-F 2 "" H 4950 6050 60  0000 C CNN
-F 3 "" H 4950 6050 60  0000 C CNN
+F 2 "pin_array_4x2" V 5050 6050 40  0001 C CNN
 	1    4950 6050
 	1    0    0    -1
@@
 F 0 "P2" H 2250 6200 50  0000 C CNN
 F 1 "CONN_3X2" V 2250 6000 40  0000 C CNN
-F 2 "" H 2250 5950 60  0000 C CNN
-F 3 "" H 2250 5950 60  0000 C CNN
+F 2 "pin_array_3x2" V 2350 6000 40  0001 C CNN
 	1    2250 5950
 	1    0    0    -1
@@
 F 0 "R2" V 2530 6400 40  0000 C CNN
 F 1 "R" V 2457 6401 40  0000 C CNN
-F 2 "" V 2380 6400 30  0000 C CNN
-F 3 "" H 2450 6400 30  0000 C CNN
+F 2 "SM0805" V 2380 6400 30  0001 C CNN
 	1    2450 6400
 	-1   0    0    1
@@
 F 0 "#PWR019" H 2450 6650 30  0001 C CNN
 F 1 "GND" H 2450 6580 30  0001 C CNN
-F 2 "" H 2450 6650 60  0000 C CNN
-F 3 "" H 2450 6650 60  0000 C CNN
 	1    2450 6650
 	1    0    0    -1

Commit message: o association of schematic->footprint.
Parts:
- P1, P2, P5, P6, P7: footprint pin_array_3x2 -> Pin_Headers:Pin_Header_Straight_2x03
- P10, P11, P12, P3, P4: footprint pin_array_4x2 -> Pin_Headers:Pin_Header_Straight_2x04
- P8, P9: footprint PIN_ARRAY_23X2 -> bumps:PIN_ARRAY_23X2
- R1, R2, R3, R4, R5: footprint SM0805 -> Resistors_SMD:Resistor_SMD0805_HandSoldering
- U1, U2, U3, U4, U5: footprint POLOLU -> bumps:POLOLU
Changed lines of the file:
@@
-EESchema Schematic File Version 2  date Sat 01 Feb 2014 09:23:24 PM PST
+EESchema Schematic File Version 2
 LIBS:power
 LIBS:device
@@
 LIBS:valves
 LIBS:BUMPS
-EELAYER 27 0
+LIBS:bumps-cache
+EELAYER 24 0
 EELAYER END
 $Descr A4 11693 8268
@@
 F 0 "U1" H 3800 4300 50  0000 C CNN
 F 1 "POLOLUSTEPPER" H 3800 4800 50  0000 C CNN
-F 2 "POLOLU" H 3850 4700 50  0001 C CNN
+F 2 "bumps:POLOLU" H 3850 4700 50  0000 C CNN
 F 3 "DOCUMENTATION" H 3800 3800 50  0001 C CNN
 	1    3800 4300
@@
 F 0 "P8" H 5300 2950 50  0000 C CNN
 F 1 "bbbp8" H 5300 3050 50  0000 C CNN
-F 2 "PIN_ARRAY_23X2" H 5300 3100 50  0001 C CNN
+F 2 "bumps:PIN_ARRAY_23X2" H 5300 3100 50  0000 C CNN
 F 3 "DOCUMENTATION" H 5300 600 50  0001 C CNN
 	1    5300 1850
@@
 F 0 "P9" H 2350 2650 50  0000 C CNN
 F 1 "bbbp9" H 2350 900 50  0000 C CNN
-F 2 "PIN_ARRAY_23X2" H 2350 2800 50  0001 C CNN
+F 2 "bumps:PIN_ARRAY_23X2" H 2350 2800 50  0000 C CNN
 F 3 "DOCUMENTATION" H 2350 350 50  0001 C CNN
 	1    2350 1700
@@
 F 0 "#PWR01" H 3650 800 30  0001 C CNN
 F 1 "GND" H 3650 730 30  0001 C CNN
+F 2 "" H 3650 800 60  0001 C CNN
+F 3 "" H 3650 800 60  0001 C CNN
 	1    3650 800
 	1    0    0    -1
@@
 F 0 "#PWR02" H 1000 800 30  0001 C CNN
 F 1 "GND" H 1000 730 30  0001 C CNN
+F 2 "" H 1000 800 60  0001 C CNN
+F 3 "" H 1000 800 60  0001 C CNN
 	1    1000 800
 	1    0    0    -1
@@
 F 0 "#PWR03" H 4550 750 30  0001 C CNN
 F 1 "GND" H 4550 680 30  0001 C CNN
+F 2 "" H 4550 750 60  0001 C CNN
+F 3 "" H 4550 750 60  0001 C CNN
 	1    4550 750
 	1    0    0    -1
@@
 F 0 "#PWR04" H 6050 750 30  0001 C CNN
 F 1 "GND" H 6050 680 30  0001 C CNN
+F 2 "" H 6050 750 60  0001 C CNN
+F 3 "" H 6050 750 60  0001 C CNN
 	1    6050 750
 	1    0    0    -1
@@
 F 0 "#PWR05" H 4550 4700 30  0001 C CNN
 F 1 "GND" H 4550 4630 30  0001 C CNN
+F 2 "" H 4550 4700 60  0001 C CNN
+F 3 "" H 4550 4700 60  0001 C CNN
 	1    4550 4700
 	1    0    0    -1
@@
 F 0 "#PWR06" H 4550 4050 30  0001 C CNN
 F 1 "GND" H 4550 3980 30  0001 C CNN
+F 2 "" H 4550 4050 60  0001 C CNN
+F 3 "" H 4550 4050 60  0001 C CNN
 	1    4550 4050
 	1    0    0    -1
@@
 F 0 "P3" H 4950 4550 50  0000 C CNN
 F 1 "CONN_4X2" V 4950 4300 40  0000 C CNN
-F 2 "pin_array_4x2" V 5050 4300 40  0001 C CNN
+F 2 "Pin_Headers:Pin_Header_Straight_2x04" V 5050 4300 40  0000 C CNN
+F 3 "" H 4950 4300 60  0001 C CNN
 	1    4950 4300
 	1    0    0    -1
@@
 F 0 "P1" H 2250 4450 50  0000 C CNN
 F 1 "CONN_3X2" V 2250 4250 40  0000 C CNN
-F 2 "pin_array_3x2" V 2350 4250 40  0001 C CNN
+F 2 "Pin_Headers:Pin_Header_Straight_2x03" V 2350 4250 40  0000 C CNN
+F 3 "" H 2250 4200 60  0001 C CNN
 	1    2250 4200
 	1    0    0    -1
@@
 F 0 "R1" V 2530 4650 40  0000 C CNN
 F 1 "R" V 2457 4651 40  0000 C CNN
-F 2 "SM0805" V 2380 4650 30  0001 C CNN
+F 2 "Resistors_SMD:Resistor_SMD0805_HandSoldering" V 2380 4650 30  0000 C CNN
+F 3 "" H 2450 4650 60  0001 C CNN
 	1    2450 4650
 	-1   0    0    1
@@
 F 0 "#PWR07" H 2450 4900 30  0001 C CNN
 F 1 "GND" H 2450 4830 30  0001 C CNN
+F 2 "" H 2450 4900 60  0001 C CNN
+F 3 "" H 2450 4900 60  0001 C CNN
 	1    2450 4900
 	1    0    0    -1
@@
 F 0 "U5" H 9200 4800 50  0000 C CNN
 F 1 "POLOLUSTEPPER" H 9200 5300 50  0000 C CNN
-F 2 "POLOLU" H 9250 5200 50  0001 C CNN
+F 2 "bumps:POLOLU" H 9250 5200 50  0000 C CNN
 F 3 "DOCUMENTATION" H 9200 4300 50  0001 C CNN
 	1    9200 4800
@@
 F 0 "#PWR08" H 9950 5200 30  0001 C CNN
 F 1 "GND" H 9950 5130 30  0001 C CNN
+F 2 "" H 9950 5200 60  0001 C CNN
+F 3 "" H 9950 5200 60  0001 C CNN
 	1    9950 5200
 	1    0    0    -1
@@
 F 0 "#PWR09" H 9950 4550 30  0001 C CNN
 F 1 "GND" H 9950 4480 30  0001 C CNN
+F 2 "" H 9950 4550 60  0001 C CNN
+F 3 "" H 9950 4550 60  0001 C CNN
 	1    9950 4550
 	1    0    0    -1
@@
 F 0 "P10" H 10350 5050 50  0000 C CNN
 F 1 "CONN_4X2" V 10350 4800 40  0000 C CNN
-F 2 "pin_array_4x2" V 10450 4800 40  0001 C CNN
+F 2 "Pin_Headers:Pin_Header_Straight_2x04" V 10450 4800 40  0000 C CNN
+F 3 "" H 10350 4800 60  0001 C CNN
 	1    10350 4800
 	1    0    0    -1
@@
 F 0 "P7" H 7650 4950 50  0000 C CNN
 F 1 "CONN_3X2" V 7650 4750 40  0000 C CNN
-F 2 "pin_array_3x2" V 7750 4750 40  0001 C CNN
+F 2 "Pin_Headers:Pin_Header_Straight_2x03" V 7750 4750 40  0000 C CNN
+F 3 "" H 7650 4700 60  0001 C CNN
 	1    7650 4700
 	1    0    0    -1
@@
 F 0 "R5" V 7930 5150 40  0000 C CNN
 F 1 "R" V 7857 5151 40  0000 C CNN
-F 2 "SM0805" V 7780 5150 30  0001 C CNN
+F 2 "Resistors_SMD:Resistor_SMD0805_HandSoldering" V 7780 5150 30  0000 C CNN
+F 3 "" H 7850 5150 60  0001 C CNN
 	1    7850 5150
 	-1   0    0    1
@@
 F 0 "#PWR010" H 7850 5400 30  0001 C CNN
 F 1 "GND" H 7850 5330 30  0001 C CNN
+F 2 "" H 7850 5400 60  0001 C CNN
+F 3 "" H 7850 5400 60  0001 C CNN
 	1    7850 5400
 	1    0    0    -1
@@
 F 0 "U3" H 9200 1550 50  0000 C CNN
 F 1 "POLOLUSTEPPER" H 9200 2050 50  0000 C CNN
-F 2 "POLOLU" H 9250 1950 50  0001 C CNN
+F 2 "bumps:POLOLU" H 9250 1950 50  0000 C CNN
 F 3 "DOCUMENTATION" H 9200 1050 50  0001 C CNN
 	1    9200 1550
@@
 F 0 "#PWR011" H 9950 1950 30  0001 C CNN
 F 1 "GND" H 9950 1880 30  0001 C CNN
+F 2 "" H 9950 1950 60  0001 C CNN
+F 3 "" H 9950 1950 60  0001 C CNN
 	1    9950 1950
 	1    0    0    -1
@@
 F 0 "#PWR012" H 9950 1300 30  0001 C CNN
 F 1 "GND" H 9950 1230 30  0001 C CNN
+F 2 "" H 9950 1300 60  0001 C CNN
+F 3 "" H 9950 1300 60  0001 C CNN
 	1    9950 1300
 	1    0    0    -1
@@
 F 0 "P11" H 10350 1800 50  0000 C CNN
 F 1 "CONN_4X2" V 10350 1550 40  0000 C CNN
-F 2 "pin_array_4x2" V 10450 1550 40  0001 C CNN
+F 2 "Pin_Headers:Pin_Header_Straight_2x04" V 10450 1550 40  0000 C CNN
+F 3 "" H 10350 1550 60  0001 C CNN
 	1    10350 1550
 	1    0    0    -1
@@
 F 0 "P5" H 7650 1700 50  0000 C CNN
 F 1 "CONN_3X2" V 7650 1500 40  0000 C CNN
-F 2 "pin_array_3x2" V 7750 1500 40  0001 C CNN
+F 2 "Pin_Headers:Pin_Header_Straight_2x03" V 7750 1500 40  0000 C CNN
+F 3 "" H 7650 1450 60  0001 C CNN
 	1    7650 1450
 	1    0    0    -1
@@
 F 0 "R3" V 7930 1900 40  0000 C CNN
 F 1 "R" V 7857 1901 40  0000 C CNN
-F 2 "SM0805" V 7780 1900 30  0001 C CNN
+F 2 "Resistors_SMD:Resistor_SMD0805_HandSoldering" V 7780 1900 30  0000 C CNN
+F 3 "" H 7850 1900 60  0001 C CNN
 	1    7850 1900
 	-1   0    0    1
@@
 F 0 "#PWR013" H 7850 2150 30  0001 C CNN
 F 1 "GND" H 7850 2080 30  0001 C CNN
+F 2 "" H 7850 2150 60  0001 C CNN
+F 3 "" H 7850 2150 60  0001 C CNN
 	1    7850 2150
 	1    0    0    -1
@@
 F 0 "U4" H 9200 3200 50  0000 C CNN
 F 1 "POLOLUSTEPPER" H 9200 3700 50  0000 C CNN
-F 2 "POLOLU" H 9250 3600 50  0001 C CNN
+F 2 "bumps:POLOLU" H 9250 3600 50  0000 C CNN
 F 3 "DOCUMENTATION" H 9200 2700 50  0001 C CNN
 	1    9200 3200
@@
 F 0 "#PWR014" H 9950 3600 30  0001 C CNN
 F 1 "GND" H 9950 3530 30  0001 C CNN
+F 2 "" H 9950 3600 60  0001 C CNN
+F 3 "" H 9950 3600 60  0001 C CNN
 	1    9950 3600
 	1    0    0    -1
@@
 F 0 "#PWR015" H 9950 2950 30  0001 C CNN
 F 1 "GND" H 9950 2880 30  0001 C CNN
+F 2 "" H 9950 2950 60  0001 C CNN
+F 3 "" H 9950 2950 60  0001 C CNN
 	1    9950 2950
 	1    0    0    -1
@@
 F 0 "P12" H 10350 3450 50  0000 C CNN
 F 1 "CONN_4X2" V 10350 3200 40  0000 C CNN
-F 2 "pin_array_4x2" V 10450 3200 40  0001 C CNN
+F 2 "Pin_Headers:Pin_Header_Straight_2x04" V 10450 3200 40  0000 C CNN
+F 3 "" H 10350 3200 60  0001 C CNN
 	1    10350 3200
 	1    0    0    -1
@@
 F 0 "P6" H 7650 3350 50  0000 C CNN
 F 1 "CONN_3X2" V 7650 3150 40  0000 C CNN
-F 2 "pin_array_3x2" V 7750 3150 40  0001 C CNN
+F 2 "Pin_Headers:Pin_Header_Straight_2x03" V 7750 3150 40  0000 C CNN
+F 3 "" H 7650 3100 60  0001 C CNN
 	1    7650 3100
 	1    0    0    -1
@@
 F 0 "R4" V 7930 3550 40  0000 C CNN
 F 1 "R" V 7857 3551 40  0000 C CNN
-F 2 "SM0805" V 7780 3550 30  0001 C CNN
+F 2 "Resistors_SMD:Resistor_SMD0805_HandSoldering" V 7780 3550 30  0000 C CNN
+F 3 "" H 7850 3550 60  0001 C CNN
 	1    7850 3550
 	-1   0    0    1
@@
 F 0 "#PWR016" H 7850 3800 30  0001 C CNN
 F 1 "GND" H 7850 3730 30  0001 C CNN
+F 2 "" H 7850 3800 60  0001 C CNN
+F 3 "" H 7850 3800 60  0001 C CNN
 	1    7850 3800
 	1    0    0    -1
@@
 F 0 "U2" H 3800 6050 50  0000 C CNN
 F 1 "POLOLUSTEPPER" H 3800 6550 50  0000 C CNN
-F 2 "POLOLU" H 3850 6450 50  0001 C CNN
+F 2 "bumps:POLOLU" H 3850 6450 50  0000 C CNN
 F 3 "DOCUMENTATION" H 3800 5550 50  0001 C CNN
 	1    3800 6050
@@
 F 0 "#PWR017" H 4550 6450 30  0001 C CNN
 F 1 "GND" H 4550 6380 30  0001 C CNN
+F 2 "" H 4550 6450 60  0001 C CNN
+F 3 "" H 4550 6450 60  0001 C CNN
 	1    4550 6450
 	1    0    0    -1
@@
 F 0 "#PWR018" H 4550 5800 30  0001 C CNN
 F 1 "GND" H 4550 5730 30  0001 C CNN
+F 2 "" H 4550 5800 60  0001 C CNN
+F 3 "" H 4550 5800 60  0001 C CNN
 	1    4550 5800
 	1    0    0    -1
@@
 F 0 "P4" H 4950 6300 50  0000 C CNN
 F 1 "CONN_4X2" V 4950 6050 40  0000 C CNN
-F 2 "pin_array_4x2" V 5050 6050 40  0001 C CNN
+F 2 "Pin_Headers:Pin_Header_Straight_2x04" V 5050 6050 40  0000 C CNN
+F 3 "" H 4950 6050 60  0001 C CNN
 	1    4950 6050
 	1    0    0    -1
@@
 F 0 "P2" H 2250 6200 50  0000 C CNN
 F 1 "CONN_3X2" V 2250 6000 40  0000 C CNN
-F 2 "pin_array_3x2" V 2350 6000 40  0001 C CNN
+F 2 "Pin_Headers:Pin_Header_Straight_2x03" V 2350 6000 40  0000 C CNN
+F 3 "" H 2250 5950 60  0001 C CNN
 	1    2250 5950
 	1    0    0    -1
@@
 F 0 "R2" V 2530 6400 40  0000 C CNN
 F 1 "R" V 2457 6401 40  0000 C CNN
-F 2 "SM0805" V 2380 6400 30  0001 C CNN
+F 2 "Resistors_SMD:Resistor_SMD0805_HandSoldering" V 2380 6400 30  0000 C CNN
+F 3 "" H 2450 6400 60  0001 C CNN
 	1    2450 6400
 	-1   0    0    1
@@
 F 0 "#PWR019" H 2450 6650 30  0001 C CNN
 F 1 "GND" H 2450 6580 30  0001 C CNN
+F 2 "" H 2450 6650 60  0001 C CNN
+F 3 "" H 2450 6650 60  0001 C CNN
 	1    2450 6650
 	1    0    0    -1

Commit message: o Add end-switches and one capacitor.
Parts:
- added C1: CAPAPOL, Capacitors_SMD:c_elec_5x5.8, symbol CAPAPOL
- added P13, P14, P15: CONN_2, Pin_Headers:Pin_Header_Straight_1x02, symbol CONN_2
Connections:
- net labels added: END_X, END_Y, END_Z
- wire segments 59 -> 64

Commit message: o Add FETs, Power Input.
Parts:
- added C2, C3, C4, C5: CAPAPOL, Capacitors_SMD:c_elec_5x5.8, symbol CAPAPOL
- added F1: FUSE, Fuse_Holders_and_Fuses:Fuse_TE5_Littlefuse-395Series, symbol FUSE
- added K1: PWM Out, symbol CONN_3
- added P16: MPower, Connect:AK300-2, symbol CONN_2
- added Q1, Q2: AOD413A, symbol MOSFET_N
- P1, P2, P5, P6, P7: value CONN_3X2 -> MicroStep
- P13: value CONN_2 -> END-X
- P14: value CONN_2 -> END-Y
- P15: value CONN_2 -> END-Z
- P8: value bbbp8 -> P8 Header
- P9: value bbbp9 -> P9 Header
Connections:
- net labels added: PWM_1, PWM_2, PWM_3, PWM_4
- wire segments 64 -> 81
Other:
- moved on the sheet: R1, R2, U1, U2

Commit message: o more generic fet name.
Parts:
- Q1, Q2: value AOD413A -> N-FET
Changed lines of the file:
@@
 P 1800 4700
 F 0 "Q2" H 1810 4870 60  0000 R CNN
-F 1 "AOD413A" H 2350 4750 60  0000 R CNN
+F 1 "N-FET" H 2350 4750 60  0000 R CNN
 F 2 "" H 1800 4700 60  0000 C CNN
 F 3 "" H 1800 4700 60  0000 C CNN
@@
 P 1800 4200
 F 0 "Q1" H 1810 4370 60  0000 R CNN
-F 1 "AOD413A" H 2350 4250 60  0000 R CNN
+F 1 "N-FET" H 2350 4250 60  0000 R CNN
 F 2 "" H 1800 4200 60  0000 C CNN
 F 3 "" H 1800 4200 60  0000 C CNN

Commit message: o Add voltage regulator: generate 5V out of motor voltage.
Parts:
- added C6: 110p, SMD_Packages:SM0805, symbol C
- added C7: CAPAPOL, Capacitors_SMD:c_elec_5x5.8, symbol CAPAPOL
- added D1: DIODESCH, SMD_Packages:SM0805, symbol DIODESCH
- added L1: 68u, Inductors:INDUCTOR_V, symbol INDUCTOR
- added R6: 1k, SMD_Packages:SM0805, symbol R
- added R7: 0R3, SMD_Packages:SM0805, symbol R
- added R8: 3k, SMD_Packages:SM0805, symbol R
- added U6: MC34063, SOIC_Packages:SOIC-8_N, symbol MC34063
- K1: footprint (none) -> Connect:PINHEAD1-3
- Q1, Q2: footprint (none) -> Transistors_TO-220:TO-220_FET-GDS_Vertical_MountedFromLS
Connections:
- net labels added: VDD_5V
- wire segments 81 -> 97
